File: hardware/synth_machine.kicad_sch (KiCad schematic)
At the start: 90 parts, among them J1 USB-C (MIDI + 5V power), J10 Pot Wave (10k lin, panel moun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, J11 Pot Attack (10k lin, panel mo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, J12 Pot Decay (10k lin, panel mou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, J13 Pot Sustain (10k lin, panel m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, J14 Pot Release (10k lin, panel m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, J3 Panel power switch, J4 From amp screw terminals (L+ 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, J5 Speaker L (JST-PH), J6 Speaker R (JST-PH), J7 Headphones 3.5mm (CUI SJ1-351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, J8 Expansion, J9 Panel LED (anode, cathode), Q1 2N3904, SW1 KEY C4 (direct D10) - 2x Keys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, SW10 D#4 [c4 r1] - 2x Keystone 3534, SW11 F#4 [c3 r1] - 2x Keystone 3534, SW12 G#4 [c2 r1] - 2x Keystone 3534, SW13 A#4 [c1 r1] - 2x Keystone 3534, SW14 BTN1 [c0 r0] - 2x Keystone 35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, SW15 BTN2 [c0 r1] - 2x Keystone 35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, SW16 BTN3 [c1 r0] - 2x Keystone 35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, SW17 BTN4 [c2 r0] - 2x Keystone 35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, SW18 BTN5 [c3 r0] - 2x Keystone 35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, SW19 BTN6 [c4 r0] - 2x Keystone 35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, SW2 D4 [c5 r1] - 2x Keystone 3534, SW3 E4 [c5 r2] - 2x Keystone 3534, SW4 F4 [c4 r2] - 2x Keystone 3534, SW5 G4 [c3 r2] - 2x Keystone 3534, SW6 A4 [c2 r2] - 2x Keystone 3534, SW7 B4 [c1 r2] - 2x Keystone 3534, SW8 C5 [c0 r2] - 2x Keystone 3534, SW9 C#4 [c5 r0] - 2x Keystone 3534, U1 Daisy Seed, U2 TPA6138A2PWR

Commit message: Drop the panel power switch and LED header; KiCad 10 compatibility
- J3 removed: the polyfuse now feeds +5V directly (unplug USB to power off)
- J9/R7 removed, D12 is free again
- USB-C shield pad is "SH" in the KiCad 10 footprint library (was S1); the
  generator maps both so the shield stays on GND
- re-routed with the locked audio pre-routes: 805 segments, 48 vias, 0 unrouted

Co-Authored-By: Claude Fable 5.1 <noreply@anthropic.com>
Parts:
- removed J3: Panel power switch, Connector_PinHeader_2.54mm:PinHeader_1x02_P2.54mm_Vertical, symbol Connector_Generic:Conn_01x02
- removed J9: Panel LED (anode, cathode), Connector_PinHeader_2.54mm:PinHeader_1x02_P2.54mm_Vertical, symbol Connector_Generic:Conn_01x02
- removed R7: 1k, Resistor_THT:R_Axial_DIN0207_L6.3mm_D2.5mm_P10.16mm_Horizontal, symbol Device:R
Connections:
- net +5V_SW is gone; now on net +5V: F1.2
- net GND: now also J1.SH (SHIELD); no longer J1.S1 (SHIELD)
- net LED: no longer names the net of U1.13 (D12)
- no-connect marks 12 -> 13
Other:
- note added: "POWER: USB-C only. VBUS -> 2A polyfuse -> +5V rail for Seed VIN and the amp. 5.1k CC pull-downs advertise a 1.5A sink."
- note removed: "POWER: USB-C only. VBUS -> 2A polyfuse -> panel switch (J3) -> +5V rail for Seed VIN and the amp. 5.1k CC pull-downs advertise a 1.5A sink."

Commit message: Put the MAX98306 on the board and prepare for JLCPCB SMT assembly
- U3 MAX98306ETD+T (TDFN-14, thermal vias) replaces the Adafruit breakout
  header A1 and the speaker return header J4; 1u input caps, 10u + 100n
  decoupling, 100k SHDN pull-up, 100k gain resistor (9 dB) and a 3-pad
  solder jumper for 12/18 dB
- amp fan-out hand-routed: 0.2 mm stubs from the 0.4 mm pitch pads, vias,
  0.3 mm B.Cu bus to the ferrite beads; speaker nets renamed to P/N so
  KiCad/Freerouting stop treating them as differential pairs
- design rules 0.2 mm track / 0.15 mm clearance / 0.2 mm min drill
- all SMD passives are 0805 with LCSC codes; CC pull-downs and the
  headphone-detect resistors moved from axial to 0805
- fab.sh emits jlcpcb_bom.csv / jlcpcb_cpl.csv for top-side assembly
- routed: 915 segments, 61 vias, 0 unrouted, DRC clean apart from known nits

Co-Authored-By: Claude Fable 5.1 <noreply@anthropic.com>
Parts:
- removed A1: Adafruit MAX98306 amp breakout, SynthMachine:Adafruit_MAX98306_Breakout, symbol Connector_Generic:Conn_01x09
- removed J4: From amp screw terminals (L+ L- R+ R-), Connector_PinHeader_2.54mm:PinHeader_1x04_P2.54mm_Vertical, symbol Connector_Generic:Conn_01x04
- added C14: 10u, Capacitor_SMD:C_0805_2012Metric, symbol Device:C
- added C15: 100n, Capacitor_SMD:C_0805_2012Metric, symbol Device:C
- added C16, C17, C18, C19: 1u, Capacitor_SMD:C_0805_2012Metric, symbol Device:C
- added JP1: GAIN: 1-2 = 18dB, open = R13, 2-3 = 12dB, Jumper:SolderJumper-3_P1.3mm_Open_RoundedPad1.0x1.5mm, symbol Jumper:SolderJumper_3_Open
- added R13, R14: 100k, Resistor_SMD:R_0805_2012Metric, symbol Device:R
- added U3: MAX98306ETD+T, Package_DFN_QFN:TDFN-14-1EP_3x3mm_P0.4mm_EP1.78x2.35mm_ThermalVias, symbol SynthMachine:MAX98306
- C10, C9: LCSC (none) -> C14857
- C11, C12, C7, C8: LCSC (none) -> C28323
- C13: value 2u2 -> 10u; LCSC (none) -> C15850
- C2, C3, C4, C5: footprint Capacitor_THT:C_Disc_D3.0mm_W1.6mm_P2.50mm -> Capacitor_SMD:C_0805_2012Metric; LCSC (none) -> C53172
- R1, R2: footprint Resistor_THT:R_Axial_DIN0207_L6.3mm_D2.5mm_P10.16mm_Horizontal -> Resistor_SMD:R_0805_2012Metric; LCSC (none) -> C27834
- R10, R11, R4, R8, R9: LCSC (none) -> C17414
- R12: LCSC (none) -> C17407
- R3: footprint Resistor_THT:R_Axial_DIN0207_L6.3mm_D2.5mm_P10.16mm_Horizontal -> Resistor_SMD:R_0805_2012Metric; LCSC (none) -> C17407
- R5, R6: footprint Resistor_THT:R_Axial_DIN0207_L6.3mm_D2.5mm_P10.16mm_Horizontal -> Resistor_SMD:R_0805_2012Metric; LCSC (none) -> C17414
- U2: LCSC (none) -> C183097
Connections:
- net +5V: now also C14.1, C15.1, JP1.3 (B), R13.2, R14.2, U3.11 (PVDD), U3.12 (PVDD)
- net AMP_SD: now also R14.1, U3.2 (~{SHDN})
- net AUDIO_L: now also C16.1
- net AUDIO_R: now also C17.1
- net GND: now also C14.2, C15.2, C18.1, C19.1, JP1.1 (A), U3.1 (PGND), U3.15 (EP), U3.8 (PGND)
- net SPKF_L+ renamed SPKF_RN
- net SPKF_RN: now also J6.2 (Pin_2); no longer J5.1 (Pin_1)
- net SPKF_L- renamed SPKF_RP
- net SPKF_RP: now also J6.1 (Pin_1); no longer J5.2 (Pin_2)
- net SPKF_R+ renamed SPKF_LP
- net SPKF_LP: now also J5.1 (Pin_1); no longer J6.1 (Pin_1)
- net SPKF_R- renamed SPKF_LN
- net SPKF_LN: now also J5.2 (Pin_2); no longer J6.2 (Pin_2)
- net SPK_L+ renamed SPK_RN
- net SPK_RN: now also U3.9 (OUTR-)
- net SPK_L- renamed SPK_RP
- net SPK_RP: now also U3.10 (OUTR+)
- net SPK_R+ renamed SPK_LP
- net SPK_LP: now also U3.13 (OUTL+)
- net SPK_R- renamed SPK_LN
- net SPK_LN: now also U3.14 (OUTL-)
- new net AMP_GAIN: JP1.2 (C), R13.1, U3.5 (GAIN)
- new net AMP_INL: C16.2, U3.3 (INL+)
- new net AMP_INLN: C18.2, U3.4 (INL-)
- new net AMP_INR: C17.2, U3.7 (INR+)
- new net AMP_INRN: C19.2, U3.6 (INR-)
- no-connect marks 13 -> 11
Other:
- note added: "AMP: MAX98306 on board, single-ended inputs (1u caps, - inputs to GND). Gain: R13 100k to PVDD = 9 dB, JP1 straps GAIN to GND (18 dB) or PVDD (12 dB). Outputs -> ferrite + 220p EMI filter -> JST-PH."
- note removed: "AMP: Adafruit #987 breakout on a 1x9 header, single-ended inputs (L-/R- to GND). Speaker outputs come back via J4 -> ferrite + 220p EMI filter -> JST-PH."

Commit message: Carrier v0.3: compact 100x100 board, JST-XH leads for buttons and pots
- Buttons no longer plug into the board: one JST-XH 2-pin header per key
  (10 down the left edge, 9 along the bottom), pots on JST-XH 3-pin headers
  down the right edge; board shrinks to 100 x 100 mm (JLC cheap tier)
- USB-C, headphone jack and the Seed's own USB all on the top edge
- Seed3 supported (same pinout/outline as the original Seed)
- more SMT for JLC: 1N4148W SOD-123 diodes, 0805 ferrite beads, MMBT3904
  SOT-23, 0805 100n; hand-solder list is now connectors, sockets, fuse, C1
- audio pre-routes reworked for the new geometry (no crossings), amp
  fan-out kept; 808 segments, 46 vias, 0 unrouted, DRC clean apart from the
  known library nits
- README rewritten; Digi-Key list rewritten for the XH connectors

Co-Authored-By: Claude Fable 5.1 <noreply@anthropic.com>
Parts:
- removed H5, H6: M3, MountingHole:MountingHole_3.2mm_M3, symbol Mechanical:MountingHole
- removed Q1: 2N3904, Package_TO_SOT_THT:TO-92_Inline, symbol Transistor_BJT:Q_NPN_EBC
- removed SW1: KEY C4 (direct D10) - 2x Keystone 3534, SynthMachine:ArcadeButton_24mm_Keystone3534, symbol Switch:SW_Push
- removed SW10: D#4 [c4 r1] - 2x Keystone 3534, SynthMachine:ArcadeButton_24mm_Keystone3534, symbol Switch:SW_Push
- removed SW11: F#4 [c3 r1] - 2x Keystone 3534, SynthMachine:ArcadeButton_24mm_Keystone3534, symbol Switch:SW_Push
- removed SW12: G#4 [c2 r1] - 2x Keystone 3534, SynthMachine:ArcadeButton_24mm_Keystone3534, symbol Switch:SW_Push
- removed SW13: A#4 [c1 r1] - 2x Keystone 3534, SynthMachine:ArcadeButton_24mm_Keystone3534, symbol Switch:SW_Push
- removed SW14: BTN1 [c0 r0] - 2x Keystone 3534, SynthMachine:ArcadeButton_24mm_Keystone3534, symbol Switch:SW_Push
- removed SW15: BTN2 [c0 r1] - 2x Keystone 3534, SynthMachine:ArcadeButton_24mm_Keystone3534, symbol Switch:SW_Push
- removed SW16: BTN3 [c1 r0] - 2x Keystone 3534, SynthMachine:ArcadeButton_24mm_Keystone3534, symbol Switch:SW_Push
- removed SW17: BTN4 [c2 r0] - 2x Keystone 3534, SynthMachine:ArcadeButton_24mm_Keystone3534, symbol Switch:SW_Push
- removed SW18: BTN5 [c3 r0] - 2x Keystone 3534, SynthMachine:ArcadeButton_24mm_Keystone3534, symbol Switch:SW_Push
- removed SW19: BTN6 [c4 r0] - 2x Keystone 3534, SynthMachine:ArcadeButton_24mm_Keystone3534, symbol Switch:SW_Push
- removed SW2: D4 [c5 r1] - 2x Keystone 3534, SynthMachine:ArcadeButton_24mm_Keystone3534, symbol Switch:SW_Push
- removed SW3: E4 [c5 r2] - 2x Keystone 3534, SynthMachine:ArcadeButton_24mm_Keystone3534, symbol Switch:SW_Push
- removed SW4: F4 [c4 r2] - 2x Keystone 3534, SynthMachine:ArcadeButton_24mm_Keystone3534, symbol Switch:SW_Push
- removed SW5: G4 [c3 r2] - 2x Keystone 3534, SynthMachine:ArcadeButton_24mm_Keystone3534, symbol Switch:SW_Push
- removed SW6: A4 [c2 r2] - 2x Keystone 3534, SynthMachine:ArcadeButton_24mm_Keystone3534, symbol Switch:SW_Push
- removed SW7: B4 [c1 r2] - 2x Keystone 3534, SynthMachine:ArcadeButton_24mm_Keystone3534, symbol Switch:SW_Push
- removed SW8: C5 [c0 r2] - 2x Keystone 3534, SynthMachine:ArcadeButton_24mm_Keystone3534, symbol Switch:SW_Push
- removed SW9: C#4 [c5 r0] - 2x Keystone 3534, SynthMachine:ArcadeButton_24mm_Keystone3534, symbol Switch:SW_Push
- added K1: KEY C4 (direct D10) JST-XH, Connector_JST:JST_XH_B2B-XH-A_1x02_P2.50mm_Vertical, symbol Connector_Generic:Conn_01x02
- added K10: A4 [c2 r2] JST-XH, Connector_JST:JST_XH_B2B-XH-A_1x02_P2.50mm_Vertical, symbol Connector_Generic:Conn_01x02
- added K11: A#4 [c1 r1] JST-XH, Connector_JST:JST_XH_B2B-XH-A_1x02_P2.50mm_Vertical, symbol Connector_Generic:Conn_01x02
- added K12: B4 [c1 r2] JST-XH, Connector_JST:JST_XH_B2B-XH-A_1x02_P2.50mm_Vertical, symbol Connector_Generic:Conn_01x02
- added K13: C5 [c0 r2] JST-XH, Connector_JST:JST_XH_B2B-XH-A_1x02_P2.50mm_Vertical, symbol Connector_Generic:Conn_01x02
- added K14: BTN1 [c0 r0] JST-XH, Connector_JST:JST_XH_B2B-XH-A_1x02_P2.50mm_Vertical, symbol Connector_Generic:Conn_01x02
- added K15: BTN2 [c0 r1] JST-XH, Connector_JST:JST_XH_B2B-XH-A_1x02_P2.50mm_Vertical, symbol Connector_Generic:Conn_01x02
- added K16: BTN3 [c1 r0] JST-XH, Connector_JST:JST_XH_B2B-XH-A_1x02_P2.50mm_Vertical, symbol Connector_Generic:Conn_01x02
- added K17: BTN4 [c2 r0] JST-XH, Connector_JST:JST_XH_B2B-XH-A_1x02_P2.50mm_Vertical, symbol Connector_Generic:Conn_01x02
- added K18: BTN5 [c3 r0] JST-XH, Connector_JST:JST_XH_B2B-XH-A_1x02_P2.50mm_Vertical, symbol Connector_Generic:Conn_01x02
- added K19: BTN6 [c4 r0] JST-XH, Connector_JST:JST_XH_B2B-XH-A_1x02_P2.50mm_Vertical, symbol Connector_Generic:Conn_01x02
- added K2: C#4 [c5 r0] JST-XH, Connector_JST:JST_XH_B2B-XH-A_1x02_P2.50mm_Vertical, symbol Connector_Generic:Conn_01x02
- added K3: D4 [c5 r1] JST-XH, Connector_JST:JST_XH_B2B-XH-A_1x02_P2.50mm_Vertical, symbol Connector_Generic:Conn_01x02
- added K4: D#4 [c4 r1] JST-XH, Connector_JST:JST_XH_B2B-XH-A_1x02_P2.50mm_Vertical, symbol Connector_Generic:Conn_01x02
- added K5: E4 [c5 r2] JST-XH, Connector_JST:JST_XH_B2B-XH-A_1x02_P2.50mm_Vertical, symbol Connector_Generic:Conn_01x02
- added K6: F4 [c4 r2] JST-XH, Connector_JST:JST_XH_B2B-XH-A_1x02_P2.50mm_Vertical, symbol Connector_Generic:Conn_01x02
- added K7: F#4 [c3 r1] JST-XH, Connector_JST:JST_XH_B2B-XH-A_1x02_P2.50mm_Vertical, symbol Connector_Generic:Conn_01x02
- added K8: G4 [c3 r2] JST-XH, Connector_JST:JST_XH_B2B-XH-A_1x02_P2.50mm_Vertical, symbol Connector_Generic:Conn_01x02
- added K9: G#4 [c2 r1] JST-XH, Connector_JST:JST_XH_B2B-XH-A_1x02_P2.50mm_Vertical, symbol Connector_Generic:Conn_01x02
- added Q1: MMBT3904, Package_TO_SOT_SMD:SOT-23, symbol Transistor_BJT:Q_NPN_BEC
- C6: footprint Capacitor_THT:C_Disc_D5.0mm_W2.5mm_P2.50mm -> Capacitor_SMD:C_0805_2012Metric; LCSC (none) -> C49678
- D1, D10, D11, D12, D13, D14, D15, D16, D17, D18, D2, D3, D4, D5, D6, D7, D8, D9: value 1N4148 -> 1N4148W; footprint Diode_THT:D_DO-35_SOD27_P7.62mm_Horizontal -> Diode_SMD:D_SOD-123; LCSC (none) -> C81598
- F1: value 2A hold PTC (MF-R200) -> MF-R250 2.5A PTC
- FB1, FB2, FB3, FB4: value 600R@100MHz -> 100R@100MHz 0805; footprint Inductor_THT:L_Axial_L5.3mm_D2.2mm_P7.62mm_Horizontal_Vishay_IM-1 -> Inductor_SMD:L_0805_2012Metric; LCSC (none) -> C1015
- J10: value Pot Wave (10k lin, panel mount) -> Pot WAV (10k lin, panel) JST-XH; footprint Connector_PinHeader_2.54mm:PinHeader_1x03_P2.54mm_Vertical -> Connector_JST:JST_XH_B3B-XH-A_1x03_P2.50mm_Vertical
- J11: value Pot Attack (10k lin, panel mount) -> Pot ATK (10k lin, panel) JST-XH; footprint Connector_PinHeader_2.54mm:PinHeader_1x03_P2.54mm_Vertical -> Connector_JST:JST_XH_B3B-XH-A_1x03_P2.50mm_Vertical
- J12: value Pot Decay (10k lin, panel mount) -> Pot DEC (10k lin, panel) JST-XH; footprint Connector_PinHeader_2.54mm:PinHeader_1x03_P2.54mm_Vertical -> Connector_JST:JST_XH_B3B-XH-A_1x03_P2.50mm_Vertical
- J13: value Pot Sustain (10k lin, panel mount) -> Pot SUS (10k lin, panel) JST-XH; footprint Connector_PinHeader_2.54mm:PinHeader_1x03_P2.54mm_Vertical -> Connector_JST:JST_XH_B3B-XH-A_1x03_P2.50mm_Vertical
- J14: value Pot Release (10k lin, panel mount) -> Pot REL (10k lin, panel) JST-XH; footprint Connector_PinHeader_2.54mm:PinHeader_1x03_P2.54mm_Vertical -> Connector_JST:JST_XH_B3B-XH-A_1x03_P2.50mm_Vertical
- R12, R13, R14, R3: LCSC C17407 -> C149504
- U1: value Daisy Seed -> Daisy Seed / Seed3
Connections:
- net AMP_SD: now also Q1.3 (C)
- net COL0: now also D12.1 (K); no longer D7.1 (K)
- net COL1: now also D10.1 (K), D11.1 (K); no longer D12.1 (K), D6.1 (K)
- net COL2: now also D8.1 (K), D9.1 (K); no longer D11.1 (K), D5.1 (K)
- net COL3: now also D6.1 (K), D7.1 (K); no longer D10.1 (K), D4.1 (K)
- net COL4: now also D5.1 (K); no longer D9.1 (K)
- net COL5: now also D4.1 (K); no longer D8.1 (K)
- net GND: now also K1.2 (Pin_2), Q1.2 (E)
- net KEY_C4: now also K1.1 (Pin_1)
- net Q1_B: now also Q1.1 (B)
- net ROW0: now also K14.1 (Pin_1), K16.1 (Pin_1), K17.1 (Pin_1), K18.1 (Pin_1), K19.1 (Pin_1), K2.1 (Pin_1)
- net ROW1: now also K11.1 (Pin_1), K15.1 (Pin_1), K3.1 (Pin_1), K4.1 (Pin_1), K7.1 (Pin_1), K9.1 (Pin_1)
- net ROW2: now also K10.1 (Pin_1), K12.1 (Pin_1), K13.1 (Pin_1), K5.1 (Pin_1), K6.1 (Pin_1), K8.1 (Pin_1)
- net SPKF_LN: now also C2.1, FB1.2; no longer C5.1, FB4.2
- net SPKF_LP: now also C3.1, FB2.2; no longer C4.1, FB3.2
- net SPKF_RN: now also C5.1, FB4.2; no longer C2.1, FB1.2
- net SPKF_RP: now also C4.1, FB3.2; no longer C3.1, FB2.2
- net SPK_LN: now also FB1.1; no longer FB4.1
- net SPK_LP: now also FB2.1; no longer FB3.1
- net SPK_RN: now also FB4.1; no longer FB1.1
- net SPK_RP: now also FB3.1; no longer FB2.1
- net at D1.2 (A): now also K2.2 (Pin_2)
- net at D11.2 (A): now also K12.2 (Pin_2)
- net at D2.2 (A): now also K3.2 (Pin_2)
- net at D16.2 (A): now also K17.2 (Pin_2)
- net at D18.2 (A): now also K19.2 (Pin_2)
- net at D9.2 (A): now also K10.2 (Pin_2)
- net at D3.2 (A): now also K4.2 (Pin_2)
- net at D15.2 (A): now also K16.2 (Pin_2)
- net at D10.2 (A): now also K11.2 (Pin_2)
- net at D4.2 (A): now also K5.2 (Pin_2)
- net at D7.2 (A): now also K8.2 (Pin_2)
- net at D6.2 (A): now also K7.2 (Pin_2)
- net at D8.2 (A): now also K9.2 (Pin_2)
- net at D5.2 (A): now also K6.2 (Pin_2)
- net at D12.2 (A): now also K13.2 (Pin_2)
- net at D14.2 (A): now also K15.2 (Pin_2)
- net at D17.2 (A): now also K18.2 (Pin_2)
- net at D13.2 (A): now also K14.2 (Pin_2)
Other:
- note added: "POTS: panel-mount 10k linear pots on JST-XH 3-pin: 1 = +3V3A, 2 = wiper -> A0..A4, 3 = AGND. KEYS: panel buttons on JST-XH 2-pin, one per key."
- note removed: "POTS: panel-mount 10k linear pots wired to 3-pin headers: 1 = +3V3A, 2 = wiper -> A0..A4, 3 = AGND."
