File: hardware/v0.4/synth_machine.kicad_sch (KiCad schematic)
At the start: 100 parts, among them J1 USB-C (MIDI + 5V power), J10 Pot VOL (10k lin, panel) JST-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, J11 Pot POT2 (10k lin, panel) JST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, J12 Pot POT3 (10k lin, panel) JST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, J13 Pot POT4 (10k lin, panel) JST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, J14 Pot POT5 (10k lin, panel) JST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, J15 STEMMA QT (I2C1), J5 Speaker L (JST-PH), J6 Speaker R (JST-PH), J7 Headphones 3.5mm (CUI SJ1-351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, J8 Expansion, J9 Display (SPI1), K1 KEY C4 (direct D10) JST-XH, K10 A4 [c2 r2] JST-XH, K11 A#4 [c1 r1] JST-XH, K12 B4 [c1 r2] JST-XH, K13 C5 [c0 r2] JST-XH, K14 BTN1 [c0 r0] JST-XH, K15 BTN2 [c0 r1] JST-XH, K16 BTN3 [c1 r0] JST-XH, K17 BTN4 [c2 r0] JST-XH, K18 BTN5 [c3 r0] JST-XH, K19 BTN6 [c4 r0] JST-XH, K2 C#4 [c5 r0] JST-XH, K3 D4 [c5 r1] JST-XH, K4 D#4 [c4 r1] JST-XH, K5 E4 [c5 r2] JST-XH, K6 F4 [c4 r2] JST-XH, K7 F#4 [c3 r1] JST-XH, K8 G4 [c3 r2] JST-XH, K9 G#4 [c2 r1] JST-XH, Q1 2N7002, Q2 2N7002, U1 Daisy Seed / Seed3, U2 TPA6138A2PWR, U3 MAX98306ETD+T, U4 USBLC6-2SC6

Commit message: Carrier v0.4: landscape board with one key row and onboard LiPo power
Rebuilt from the two remaining next-revision ideas (the RGB LED one is
dropped):

- 160 x 74 mm outline. All 19 key headers in one row along the bottom
  edge in panel order, rotated for a 7 mm pitch (132 mm wide), diode above
  each header and the key name below it. Pots stacked up the right edge,
  EXP and DISP headers along the top, mounting holes in the corners.
- Battery: BQ24074 charger with power path (1.5 A input limit via R19,
  0.5 A charge via R18, default timers, TS 10k), TPS61023 boost to 5.1 V
  (750k/100k, 1 uH XEL4030, 10 uF in, 2 x 22 uF out + C1), JST-PH cell on
  J17, panel power switch on J16 driving the boost's EN (JP2 bridges it),
  VBAT/2 to A10, ~CHG to A5, ~PGOOD to A11. Rails: VBUS -> F1 -> VUSB ->
  charger -> VSYS -> boost -> +5V.
- Generator: mpn/dnp per part kept; pre-routes added for the boost's
  SOT-563 pins, the output-cap link, the switch pull-up rail and nine GND
  stitching vias; battery rails in the 0.4 mm class, 0.15 mm clearance so
  0.5 mm pitch pads pass DRC.
- Routed (Freerouting 2.4.1): DRC 0 unconnected, ERC clean; fab.sh's
  PCBWay BOM now lists every fitted part.
- Docs: v0.4 README rewritten with the power section, pin map, headers and
  pre-order checks; NEXT_REVISION marks the key row and LiPo as done and
  drops the LED note; Digi-Key list adds the switch, battery and PH parts.

Co-Authored-By: Claude Fable 5.1 <noreply@anthropic.com>
Claude-Session: https://claude.ai/code/session_019ZDGV5fm4G7LwUwRWHEiwx
Parts:
- removed J8: Expansion, Connector_PinHeader_2.54mm:PinHeader_1x10_P2.54mm_Vertical, symbol Connector_Generic:Conn_01x10
- added C20: 1u, Capacitor_SMD:C_0805_2012Metric, symbol Device:C
- added C21, C22, C23: 10u, Capacitor_SMD:C_0805_2012Metric, symbol Device:C
- added C24, C25: 22u 25V, Capacitor_SMD:C_1210_3225Metric, symbol Device:C
- added C26: 100n, Capacitor_SMD:C_0805_2012Metric, symbol Device:C
- added J16: Power switch (panel SPST) JST-XH, Connector_JST:JST_XH_B2B-XH-A_1x02_P2.50mm_Vertical, symbol Connector_Generic:Conn_01x02
- added J17: Battery 1S LiPo (JST-PH, 1 = +), Connector_JST:JST_PH_B2B-PH-K_1x02_P2.00mm_Vertical, symbol Connector_Generic:Conn_01x02
- added J8: Expansion, Connector_PinHeader_2.54mm:PinHeader_1x08_P2.54mm_Vertical, symbol Connector_Generic:Conn_01x08
- added JP2: always on (bridges the power switch), Jumper:SolderJumper-2_P1.3mm_Open_RoundedPad1.0x1.5mm, symbol Jumper:SolderJumper_2_Open
- added L1: 1u 4x4 (XEL4030-102ME), Inductor_SMD:L_Coilcraft_XxL4030, symbol Device:L
- added R18: 1k8 (ISET 0.5A), Resistor_SMD:R_0805_2012Metric, symbol Device:R
- added R19: 1k1 (ILIM 1.5A), Resistor_SMD:R_0805_2012Metric, symbol Device:R
- added R20, R28: 10k, Resistor_SMD:R_0805_2012Metric, symbol Device:R
- added R21, R22, R23, R24, R26, R27: 100k, Resistor_SMD:R_0805_2012Metric, symbol Device:R
- added R25: 750k (FB, 5.1V), Resistor_SMD:R_0805_2012Metric, symbol Device:R
- added U5: BQ24074RGTR, Package_DFN_QFN:VQFN-16-1EP_3x3mm_P0.5mm_EP1.6x1.6mm_ThermalVias, symbol Battery_Management:BQ24074RGT
- added U6: TPS61023DRLR, Package_TO_SOT_SMD:SOT-563, symbol SynthMachine:TPS61023
Connections:
- net +3V3: now also J8.6 (Pin_6), R21.1, R22.1
- net +5V: now also C24.1, C25.1, J8.7 (Pin_7), R25.1, U6.6 (VOUT); no longer F1.2
- net EXP_A6: now also J8.2 (Pin_2)
- net GND: now also C20.2, C21.2, C22.2, C23.2, C24.2, C25.2, C26.2, J17.2 (Pin_2), J8.8 (Pin_8), R18.2, R19.2, R20.2, R24.2, R26.2, R27.2, U5.17 (VSS), U5.4 (~{CE}), U5.6 (EN1), U5.8 (VSS), U6.4 (GND)
- net HP_DET: now also J8.3 (Pin_3)
- net HP_MUTE: now also J8.1 (Pin_1)
- net MUTE: now also J8.4 (Pin_4)
- net EXP_A10 renamed VBAT_SENSE
- net VBAT_SENSE: now also C26.1, R23.2, R24.1
- net EXP_A11 renamed USB_PGOOD
- net USB_PGOOD: now also R21.2, U5.7 (~{PGOOD})
- net EXP_A5 renamed CHG_STAT
- net CHG_STAT: now also R22.2, U5.9 (~{CHG})
- new net BOOST_EN: J16.2 (Pin_2), JP2.2 (B), R27.1, U6.2 (EN)
- new net BOOST_FB: R25.2, R26.1, U6.1 (FB)
- new net BOOST_SW: L1.2, U6.5 (SW)
- new net ILIM: R19.1, U5.12 (ILIM)
- new net ISET: R18.1, U5.16 (ISET)
- new net SW_HI: J16.1 (Pin_1), JP2.1 (A), R28.2
- new net TS: R20.1, U5.1 (TS)
- new net VBAT: C22.1, J17.1 (Pin_1), R23.1, U5.2 (BAT), U5.3 (BAT)
- new net VSYS: C21.1, C23.1, J8.5 (Pin_5), L1.1, R28.1, U5.10 (OUT), U5.11 (OUT), U5.5 (EN2), U6.3 (VIN)
- new net VUSB: C20.1, F1.2, U5.13 (IN)
- no-connect marks 6 -> 8
Other:
- note added: "BATTERY: BQ24074, EN2=1/EN1=0 -> 1.5A input limit (R19), 0.5A charge (R18), default timers, 10% termination, TS = 10k. VSYS = 4.4V on USB, else VBAT. ~CHG -> A5, ~PGOOD -> A11 (100k pull-ups). VBAT/2 -> A10."
- note added: "BOOST: TPS61023 5.1V (750k/100k), 1uH, 10uF in, 2x22uF out + C1. EN from the panel switch on J16 (or JP2 bridged) via R28, R27 pull-down = off. Use a protected LiPo cell; J17 pin 1 = +."
- note added: "POWER: VBUS -> F1 2.5A PTC -> VUSB -> U5 charger (power path) -> VSYS -> U6 boost -> +5V for Seed VIN and the amp. 5.1k CC pull-downs advertise a 1.5A sink. U4 = ESD on D+/D-."
- note removed: "POWER: USB-C only. VBUS -> 2.5A SMD polyfuse -> +5V rail for Seed VIN and the amp. 5.1k CC pull-downs advertise a 1.5A sink. U4 = ESD on D+/D-."

Commit message: Carrier v0.4: bank pots replaced by I2C encoders; volume pot only
J11..J14 are gone. J10 (volume, A0) stays on the right edge; the four bank
controls are seesaw rotary encoders on J15 (STEMMA QT, I2C1), now placed
mid-height on the right edge. A1/A2/A4/A9 go to the expansion header,
which grows to 1x12; DISP moves right to make room.

Pre-routes added for the charger's OUT and EN2 pins (0.5 mm pitch QFN) so
the VSYS rail always completes. Routed: DRC 0 unconnected, ERC clean.

Firmware HW=carrier4: reads A0 only and leaves the bank inputs alone (they
float without pots); encoder support is still to come. Docs, Digi-Key list
and NEXT_REVISION updated; the encoder item is marked done in hardware.

Co-Authored-By: Claude Fable 5.1 <noreply@anthropic.com>
Claude-Session: https://claude.ai/code/session_019ZDGV5fm4G7LwUwRWHEiwx
Parts:
- removed J11: Pot POT2 (10k lin, panel) JST-XH, Connector_JST:JST_XH_B3B-XH-A_1x03_P2.50mm_Vertical, symbol Connector_Generic:Conn_01x03
- removed J12: Pot POT3 (10k lin, panel) JST-XH, Connector_JST:JST_XH_B3B-XH-A_1x03_P2.50mm_Vertical, symbol Connector_Generic:Conn_01x03
- removed J13: Pot POT4 (10k lin, panel) JST-XH, Connector_JST:JST_XH_B3B-XH-A_1x03_P2.50mm_Vertical, symbol Connector_Generic:Conn_01x03
- removed J14: Pot POT5 (10k lin, panel) JST-XH, Connector_JST:JST_XH_B3B-XH-A_1x03_P2.50mm_Vertical, symbol Connector_Generic:Conn_01x03
- removed J8: Expansion, Connector_PinHeader_2.54mm:PinHeader_1x08_P2.54mm_Vertical, symbol Connector_Generic:Conn_01x08
- added J8: Expansion, Connector_PinHeader_2.54mm:PinHeader_1x12_P2.54mm_Vertical, symbol Connector_Generic:Conn_01x12
Connections:
- net +3V3: now also J8.10 (Pin_10)
- net +5V: now also J8.11 (Pin_11)
- net EXP_A6: now also J8.5 (Pin_5)
- net GND: now also J8.12 (Pin_12)
- net HP_DET: now also J8.7 (Pin_7)
- net HP_MUTE: now also J8.1 (Pin_1)
- net MUTE: now also J8.8 (Pin_8)
- net VSYS: now also J8.9 (Pin_9)
- net POT_2 renamed EXP_A1
- net EXP_A1: now also J8.2 (Pin_2)
- net POT_3 renamed EXP_A2
- net EXP_A2: now also J8.3 (Pin_3)
- net POT_4 renamed EXP_A9
- net EXP_A9: now also J8.6 (Pin_6)
- net POT_5 renamed EXP_A4
- net EXP_A4: now also J8.4 (Pin_4)
Other:
- note added: "POT: master volume, 10k linear on JST-XH 3-pin: 1 = +3V3A, 2 = wiper -> A0, 3 = AGND. The four bank controls are I2C encoders on J15. KEYS: panel buttons on JST-XH 2-pin, one per key."
- note removed: "POTS: panel-mount 10k linear pots on JST-XH 3-pin: 1 = +3V3A, 2 = wiper, 3 = AGND. VOL = A0, POT2 = A1, POT3 = A2, POT4 = A9, POT5 = A4. KEYS: panel buttons on JST-XH 2-pin, one per key."

Commit message: Carrier v0.4: top-entry STEMMA QT at the top right, volume header on the left edge, jack 1.5 mm proud
- J15 becomes the vertical JST SH (BM04B-SRSS-TB, LCSC C160390) at the top
  right so the encoder cable leaves upward toward the panel; the DNP
  pull-ups follow it. Top-right mounting hole back at (155, 4).
- J10 (volume pot) moves to the left edge under the USB-C, matching where
  the pot sits on the panel.
- J7 headphone jack moved 1.5 mm toward the top edge; its nose now stands
  proud of the board edge instead of flush.
- One more pre-route (FB divider to +5V) so the boost cluster routes every
  time. DRC 0 unconnected, ERC clean.
- README: connector table, J15 pin-1 check, note that F1 and L1 only look
  empty in the render because KiCad has no 3D models for those footprints.

Co-Authored-By: Claude Fable 5.1 <noreply@anthropic.com>
Claude-Session: https://claude.ai/code/session_019ZDGV5fm4G7LwUwRWHEiwx
Parts:
- J15: footprint Connector_JST:JST_SH_SM04B-SRSS-TB_1x04-1MP_P1.00mm_Horizontal -> Connector_JST:JST_SH_BM04B-SRSS-TB_1x04-1MP_P1.00mm_Vertical; LCSC C160404 -> C160390; MPN SM04B-SRSS-TB(LF)(SN) -> BM04B-SRSS-TB(LF)(SN)

Commit message: Carrier v0.4: peripheral 3.3 V rail (AP7361C-33) for encoders, display and EXP
U7, a 1 A SOT-223 LDO on +5V, makes 3V3P for the STEMMA QT connector, the
display header, the expansion header's 3V3 pin and the DNP I2C pull-ups.
The Seed's regulator now carries only the Seed, the headphone amp and the
pull-ups, so the encoder boards' NeoPixels can no longer sag it. Pinout
(1 IN, 2 GND tab, 3 OUT) checked against the AP7361C datasheet's SOT223
column; 10 uF each side placed against the footprint's stacked pins; +5V
pre-routed from the trunk to the input pin and cap, 3V3P to the output
cap. Routed: DRC 0 unconnected, ERC clean. README power section and
header tables updated.

Co-Authored-By: Claude Fable 5.1 <noreply@anthropic.com>
Claude-Session: https://claude.ai/code/session_019ZDGV5fm4G7LwUwRWHEiwx
Parts:
- added C27, C28: 10u, Capacitor_SMD:C_0805_2012Metric, symbol Device:C
- added U7: AP7361C-33E-13, Package_TO_SOT_SMD:SOT-223-3_TabPin2, symbol Regulator_Linear:SPX2920M3-3.3_SOT223
Connections:
- net +3V3: no longer J15.2 (Pin_2), J8.10 (Pin_10), J9.2 (Pin_2), R16.1, R17.1
- net +5V: now also C27.1, U7.1 (VI)
- net GND: now also C27.2, C28.2, U7.2 (GND)
- new net +3V3P: C28.1, J15.2 (Pin_2), J8.10 (Pin_10), J9.2 (Pin_2), R16.1, R17.1, U7.3 (VO)
Other:
- note added: "3V3P: AP7361C-33 LDO from +5V feeds the encoders (J15), the display (J9) and J8's 3V3 pin, so the Seed's regulator only carries the Seed, the headphone amp and pull-ups."
