File: hardware/v0.4/synth_machine.kicad_sch (KiCad schematic)
At the start: 123 parts, among them J1 USB-C (MIDI + 5V power), J10 Pot VOL (10k lin, panel) JST-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, J15 STEMMA QT (I2C1), J16 Power switch (panel SPST) JST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, J17 Battery 1S LiPo (JST-PH, 1 = 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, J5 Speaker L (JST-PH), J6 Speaker R (JST-PH), J7 Headphones 3.5mm (CUI SJ1-351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, J8 Expansion, J9 Display (SPI1), K1 KEY C4 (direct D10) JST-XH, K10 A4 [c2 r2] JST-XH, K11 A#4 [c1 r1] JST-XH, K12 B4 [c1 r2] JST-XH, K13 C5 [c0 r2] JST-XH, K14 BTN1 [c0 r0] JST-XH, K15 BTN2 [c0 r1] JST-XH, K16 BTN3 [c1 r0] JST-XH, K17 BTN4 [c2 r0] JST-XH, K18 BTN5 [c3 r0] JST-XH, K19 BTN6 [c4 r0] JST-XH, K2 C#4 [c5 r0] JST-XH, K3 D4 [c5 r1] JST-XH, K4 D#4 [c4 r1] JST-XH, K5 E4 [c5 r2] JST-XH, K6 F4 [c4 r2] JST-XH, K7 F#4 [c3 r1] JST-XH, K8 G4 [c3 r2] JST-XH, K9 G#4 [c2 r1] JST-XH, Q1 2N7002, Q2 2N7002, U1 Daisy Seed / Seed3, U2 TPA6138A2PWR, U3 MAX98306ETD+T, U4 USBLC6-2SC6, U5 BQ24074RGTR, U6 TPS61023DRLR, U7 AP7361C-33E-13

Commit message: Carrier v0.4: USB-C receptacle is the HRO TYPE-C-31-M-12 (in stock at JLCPCB)
The GCT USB4105-GF-A went out of stock at LCSC. The HRO part has the
same shell holes and pad pitch (pad row 0.36 mm further in) and the same
body depth, so J1 keeps its place on the top edge; KiCad's footprint for
it is used, so the pads match the part exactly. LCSC C165948, a JLCPCB
basic part. F1 moved 1.5 mm to clear the slightly larger courtyard.
Re-routed: DRC 0 unconnected, ERC clean. Gerbers, BOM and CPL regenerated.

Co-Authored-By: Claude Fable 5.1 <noreply@anthropic.com>
Claude-Session: https://claude.ai/code/session_019ZDGV5fm4G7LwUwRWHEiwx
Parts:
- J1: footprint Connector_USB:USB_C_Receptacle_GCT_USB4105-xx-A_16P_TopMnt_Horizontal -> Connector_USB:USB_C_Receptacle_HRO_TYPE-C-31-M-12; LCSC C3020560 -> C165948; MPN USB4105-GF-A -> TYPE-C-31-M-12

Commit message: Carrier v0.4: JST headers and sockets placed by JLCPCB standard assembly
LCSC numbers on the 19 key headers, the volume and switch headers (JST XH
C158012 / C144394) and the speaker and battery sockets (JST PH C131337);
the JLCPCB placement export now includes through-hole parts. README and
Digi-Key list say which parts remain hand-fitted.

Co-Authored-By: Claude Fable 5.1 <noreply@anthropic.com>
Claude-Session: https://claude.ai/code/session_019ZDGV5fm4G7LwUwRWHEiwx
Parts:
- J10: LCSC (none) -> C144394
- J16, K1, K10, K11, K12, K13, K14, K15, K16, K17, K18, K19, K2, K3, K4, K5, K6, K7, K8, K9: LCSC (none) -> C158012
- J17, J5, J6: LCSC (none) -> C131337
